File: hardware/hardware.kicad_pcb (KiCad board)
At the start: 2 copper layers, 18.5 x 108.5 mm, 56 parts, among them J1 RUN_OUT, J2 USB_C_Receptacle_USB2.0, J3 MIDI IN, J4 MIDI OUT, J5 Eurorack_Power, J6 CV1, J7 CV2, J8 CV3, J9 CV4, Q1 NPN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

Commit message: ready for fab
Parts:
- moved R10 6.71 mm to (132.3, 130.6)
- moved R9 6.14 mm to (135.9, 130.3), turned to 90 degrees
- moved D2 5.40 mm to (131.1, 134.6), turned to 90 degrees
- moved D1 1.95 mm to (130.3, 107.0), turned to 0 degrees
- moved R8 0.63 mm to (142.2, 130.8)
- moved TP3 0.57 mm to (131.8, 75.7)
- moved U2 0.51 mm to (138.4, 137.7)
- moved R1 0.36 mm to (131.3, 146.1)
- moved U4 0.25 mm to (142.0, 65.5)
- moved R2 0.24 mm to (131.3, 148.3)
Connections:
- U1 pad 13: unconnected-(U1-D9-Pad13) -> Net-(D1-A)
- U1 pad 23: unconnected-(U1-SCK/18-Pad23) -> RUN
Routing:
- net GND: track 9.69 -> 45.4 mm, vias 0 -> 6
- net Net-(D2-K): track 14.2 -> 35.0 mm, vias 0 -> 1
- net RX: track 7.16 -> 21.8 mm
- net Net-(D1-A): track 0.00 -> 7.61 mm
- net +3.3V: track 38.7 -> 31.8 mm
- net MIDVREF: track 83.7 -> 90.5 mm
- net RUN: track 12.3 -> 6.35 mm
- net Net-(J4-PadR): track 2.95 -> 8.18 mm
- net Net-(J4-PadT): track 3.63 -> 6.69 mm
- net +5V: track 36.2 -> 38.3 mm, vias 0 -> 1
- net Net-(D2-A): track 6.41 -> 4.49 mm
- net Net-(D1-K): track 2.67 -> 3.98 mm
- net Net-(J1-Tip): track 2.31 -> 3.30 mm
- net +12V: track 65.6 -> 66.1 mm
- added copper zone on B.Cu, net GND
- added copper zone on F.Cu, net GND
